Commit message: [koch_description] Rename to koch_description

File: koch_description/urdf/koch.urdf (robot description, URDF)
Before this commit: robot low_cost_robot, 7 links, 6 joints
Links:
- link base_link: geometry collision mesh filename=file://$(find koch_description)/meshes/base_link.stl scale=0.001 0.001 0.001; visual mesh filename=file://$(find koch_description)/meshes/base_link.stl scale=0.001 0.001 0.001
- link gripper_moving_1: geometry collision mesh filename=file://$(find koch_description)/meshes/gripper_moving_1.stl scale=0.001 0.001 0.001; visual mesh filename=file://$(find koch_description)/meshes/gripper_moving_1.stl scale=0.001 0.001 0.001
- link gripper_static_1: geometry collision mesh filename=file://$(find koch_description)/meshes/gripper_static_1.stl scale=0.001 0.001 0.001; visual mesh filename=file://$(find koch_description)/meshes/gripper_static_1.stl scale=0.001 0.001 0.001
- link link1_1: geometry collision mesh filename=file://$(find koch_description)/meshes/link1_1.stl scale=0.001 0.001 0.001; visual mesh filename=file://$(find koch_description)/meshes/link1_1.stl scale=0.001 0.001 0.001
- link link2_1: geometry collision mesh filename=file://$(find koch_description)/meshes/link2_1.stl scale=0.001 0.001 0.001; visual mesh filename=file://$(find koch_description)/meshes/link2_1.stl scale=0.001 0.001 0.001
- link link3_1: geometry collision mesh filename=file://$(find koch_description)/meshes/link3_1.stl scale=0.001 0.001 0.001; visual mesh filename=file://$(find koch_description)/meshes/link3_1.stl scale=0.001 0.001 0.001
- link link4_1: geometry collision mesh filename=file://$(find koch_description)/meshes/link4_1.stl scale=0.001 0.001 0.001; visual mesh filename=file://$(find koch_description)/meshes/link4_1.stl scale=0.001 0.001 0.001

File: koch_description/urdf/koch.xacro (robot description, xacro)
@@ -1,7 +1,7 @@
 <?xml version="1.0" ?>
-<robot name="low_cost_robot" xmlns:xacro="http://www.ros.org/wiki/xacro">
-<xacro:include filename="$(find low_cost_robot_description)/urdf/materials.xacro" />
-<xacro:include filename="$(find low_cost_robot_description)/urdf/low_cost_robot.trans" />
-<xacro:include filename="$(find low_cost_robot_description)/urdf/low_cost_robot.gazebo" />
+<robot name="koch" xmlns:xacro="http://www.ros.org/wiki/xacro">
+<xacro:include filename="$(find koch_description)/urdf/materials.xacro" />
+<xacro:include filename="$(find koch_description)/urdf/koch.trans" />
+<xacro:include filename="$(find koch_description)/urdf/koch.gazebo" />
 <link name="base_link">
   <inertial>
@@ -13,5 +13,5 @@
     <origin xyz="0 0 0" rpy="0 0 0"/>
     <geometry>
-      <mesh filename="file://$(find low_cost_robot_description)/meshes/base_link.stl" scale="0.001 0.001 0.001"/>
+      <mesh filename="file://$(find koch_description)/meshes/base_link.stl" scale="0.001 0.001 0.001"/>
     </geometry>
     <material name="silver"/>
@@ -20,5 +20,5 @@
     <origin xyz="0 0 0" rpy="0 0 0"/>
     <geometry>
-      <mesh filename="file://$(find low_cost_robot_description)/meshes/base_link.stl" scale="0.001 0.001 0.001"/>
+      <mesh filename="file://$(find koch_description)/meshes/base_link.stl" scale="0.001 0.001 0.001"/>
     </geometry>
   </collision>
@@ -33,5 +33,5 @@
     <origin xyz="-0.0 -0.0 -0.039" rpy="0 0 0"/>
     <geometry>
-      <mesh filename="file://$(find low_cost_robot_description)/meshes/link1_1.stl" scale="0.001 0.001 0.001"/>
+      <mesh filename="file://$(find koch_description)/meshes/link1_1.stl" scale="0.001 0.001 0.001"/>
     </geometry>
     <material name="silver"/>
@@ -40,5 +40,5 @@
     <origin xyz="-0.0 -0.0 -0.039" rpy="0 0 0"/>
     <geometry>
-      <mesh filename="file://$(find low_cost_robot_description)/meshes/link1_1.stl" scale="0.001 0.001 0.001"/>
+      <mesh filename="file://$(find koch_description)/meshes/link1_1.stl" scale="0.001 0.001 0.001"/>
     </geometry>
   </collision>
@@ -53,5 +53,5 @@
     <origin xyz="0.0002 0.0 -0.0563" rpy="0 0 0"/>
     <geometry>
-      <mesh filename="file://$(find low_cost_robot_description)/meshes/link2_1.stl" scale="0.001 0.001 0.001"/>
+      <mesh filename="file://$(find koch_description)/meshes/link2_1.stl" scale="0.001 0.001 0.001"/>
     </geometry>
     <material name="silver"/>
@@ -60,5 +60,5 @@
     <origin xyz="0.0002 0.0 -0.0563" rpy="0 0 0"/>
     <geometry>
-      <mesh filename="file://$(find low_cost_robot_description)/meshes/link2_1.stl" scale="0.001 0.001 0.001"/>
+      <mesh filename="file://$(find koch_description)/meshes/link2_1.stl" scale="0.001 0.001 0.001"/>
     </geometry>
   </collision>
@@ -73,5 +73,5 @@
     <origin xyz="-5e-05 -0.014791 -0.164647" rpy="0 0 0"/>
     <geometry>
-      <mesh filename="file://$(find low_cost_robot_description)/meshes/link3_1.stl" scale="0.001 0.001 0.001"/>
+      <mesh filename="file://$(find koch_description)/meshes/link3_1.stl" scale="0.001 0.001 0.001"/>
     </geometry>
     <material name="silver"/>
@@ -80,5 +80,5 @@
     <origin xyz="-5e-05 -0.014791 -0.164647" rpy="0 0 0"/>
     <geometry>
-      <mesh filename="file://$(find low_cost_robot_description)/meshes/link3_1.stl" scale="0.001 0.001 0.001"/>
+      <mesh filename="file://$(find koch_description)/meshes/link3_1.stl" scale="0.001 0.001 0.001"/>
     </geometry>
   </collision>
@@ -93,5 +93,5 @@
     <origin xyz="-0.000175 -0.105258 -0.167394" rpy="0 0 0"/>
     <geometry>
-      <mesh filename="file://$(find low_cost_robot_description)/meshes/link4_1.stl" scale="0.001 0.001 0.001"/>
+      <mesh filename="file://$(find koch_description)/meshes/link4_1.stl" scale="0.001 0.001 0.001"/>
     </geometry>
     <material name="silver"/>
@@ -100,5 +100,5 @@
     <origin xyz="-0.000175 -0.105258 -0.167394" rpy="0 0 0"/>
     <geometry>
-      <mesh filename="file://$(find low_cost_robot_description)/meshes/link4_1.stl" scale="0.001 0.001 0.001"/>
+      <mesh filename="file://$(find koch_description)/meshes/link4_1.stl" scale="0.001 0.001 0.001"/>
     </geometry>
   </collision>
@@ -113,5 +113,5 @@
     <origin xyz="-0.001528 -0.105265 -0.122394" rpy="0 0 0"/>
     <geometry>
-      <mesh filename="file://$(find low_cost_robot_description)/meshes/gripper_static_1.stl" scale="0.001 0.001 0.001"/>
+      <mesh filename="file://$(find koch_description)/meshes/gripper_static_1.stl" scale="0.001 0.001 0.001"/>
     </geometry>
     <material name="silver"/>
@@ -120,5 +120,5 @@
     <origin xyz="-0.001528 -0.105265 -0.122394" rpy="0 0 0"/>
     <geometry>
-      <mesh filename="file://$(find low_cost_robot_description)/meshes/gripper_static_1.stl" scale="0.001 0.001 0.001"/>
+      <mesh filename="file://$(find koch_description)/meshes/gripper_static_1.stl" scale="0.001 0.001 0.001"/>
     </geometry>
   </collision>
@@ -133,5 +133,5 @@
     <origin xyz="0.005872 -0.105015 -0.109244" rpy="0 0 0"/>
     <geometry>
-      <mesh filename="file://$(find low_cost_robot_description)/meshes/gripper_moving_1.stl" scale="0.001 0.001 0.001"/>
+      <mesh filename="file://$(find koch_description)/meshes/gripper_moving_1.stl" scale="0.001 0.001 0.001"/>
     </geometry>
     <material name="silver"/>
@@ -140,5 +140,5 @@
     <origin xyz="0.005872 -0.105015 -0.109244" rpy="0 0 0"/>
     <geometry>
-      <mesh filename="file://$(find low_cost_robot_description)/meshes/gripper_moving_1.stl" scale="0.001 0.001 0.001"/>
+      <mesh filename="file://$(find koch_description)/meshes/gripper_moving_1.stl" scale="0.001 0.001 0.001"/>
     </geometry>
   </collision>

File: koch_description/urdf/materials.xacro (robot description, xacro)
@@ -1,4 +1,4 @@
 <?xml version="1.0" ?>
-<robot name="low_cost_robot" xmlns:xacro="http://www.ros.org/wiki/xacro" >
+<robot name="koch" xmlns:xacro="http://www.ros.org/wiki/xacro" >
 <material name="silver">
   <color rgba="0.700 0.700 0.700 1.000"/>
