Commit message: [koch_description] Support ros2_control

File: koch_description/urdf/koch.xacro (robot description, xacro)
@@ -1,182 +1,238 @@
 <?xml version="1.0" ?>
 <robot name="koch" xmlns:xacro="http://www.ros.org/wiki/xacro">
-<xacro:include filename="$(find koch_description)/urdf/materials.xacro" />
-<xacro:include filename="$(find koch_description)/urdf/koch.trans" />
-<xacro:include filename="$(find koch_description)/urdf/koch.gazebo" />
-<link name="base_link">
-  <inertial>
-    <origin xyz="-0.00017023202404845418 -0.021341439639662032 0.014423161616418092" rpy="0 0 0"/>
-    <mass value="0.5164575020815119"/>
-    <inertia ixx="0.000304" iyy="0.000283" izz="0.000441" ixy="-2e-06" iyz="-6.2e-05" ixz="-1e-06"/>
-  </inertial>
-  <visual>
-    <origin xyz="0 0 0" rpy="0 0 0"/>
-    <geometry>
-      <mesh filename="file://$(find koch_description)/meshes/base_link.stl" scale="0.001 0.001 0.001"/>
-    </geometry>
-    <material name="silver"/>
-  </visual>
-  <collision>
-    <origin xyz="0 0 0" rpy="0 0 0"/>
-    <geometry>
-      <mesh filename="file://$(find koch_description)/meshes/base_link.stl" scale="0.001 0.001 0.001"/>
-    </geometry>
-  </collision>
-</link>
-<link name="link1_1">
-  <inertial>
-    <origin xyz="-0.0006216635769899589 -0.011914175885676576 0.015400174574576098" rpy="0 0 0"/>
-    <mass value="0.3956063453928257"/>
-    <inertia ixx="0.000112" iyy="7.5e-05" izz="0.000123" ixy="0.0" iyz="-1e-06" ixz="0.0"/>
-  </inertial>
-  <visual>
-    <origin xyz="-0.0 -0.0 -0.039" rpy="0 0 0"/>
-    <geometry>
-      <mesh filename="file://$(find koch_description)/meshes/link1_1.stl" scale="0.001 0.001 0.001"/>
-    </geometry>
-    <material name="silver"/>
-  </visual>
-  <collision>
-    <origin xyz="-0.0 -0.0 -0.039" rpy="0 0 0"/>
-    <geometry>
-      <mesh filename="file://$(find koch_description)/meshes/link1_1.stl" scale="0.001 0.001 0.001"/>
-    </geometry>
-  </collision>
-</link>
-<link name="link2_1">
-  <inertial>
-    <origin xyz="0.00015778948024297947 -0.0012168309893684582 0.07161179945761596" rpy="0 0 0"/>
-    <mass value="0.3916070272991037"/>
-    <inertia ixx="0.00052" iyy="0.000534" izz="8.4e-05" ixy="-1e-06" iyz="-3.7e-05" ixz="-2e-06"/>
-  </inertial>
-  <visual>
-    <origin xyz="0.0002 0.0 -0.0563" rpy="0 0 0"/>
-    <geometry>
-      <mesh filename="file://$(find koch_description)/meshes/link2_1.stl" scale="0.001 0.001 0.001"/>
-    </geometry>
-    <material name="silver"/>
-  </visual>
-  <collision>
-    <origin xyz="0.0002 0.0 -0.0563" rpy="0 0 0"/>
-    <geometry>
-      <mesh filename="file://$(find koch_description)/meshes/link2_1.stl" scale="0.001 0.001 0.001"/>
-    </geometry>
-  </collision>
-</link>
-<link name="link3_1">
-  <inertial>
-    <origin xyz="7.243666489899892e-05 0.05069893196527342 0.002850799344132765" rpy="0 0 0"/>
-    <mass value="0.4404689720232285"/>
-    <inertia ixx="0.000302" iyy="5.5e-05" izz="0.000322" ixy="-1e-06" iyz="-0.0" ixz="0.0"/>
-  </inertial>
-  <visual>
-    <origin xyz="-5e-05 -0.014791 -0.164647" rpy="0 0 0"/>
-    <geometry>
-      <mesh filename="file://$(find koch_description)/meshes/link3_1.stl" scale="0.001 0.001 0.001"/>
-    </geometry>
-    <material name="silver"/>
-  </visual>
-  <collision>
-    <origin xyz="-5e-05 -0.014791 -0.164647" rpy="0 0 0"/>
-    <geometry>
-      <mesh filename="file://$(find koch_description)/meshes/link3_1.stl" scale="0.001 0.001 0.001"/>
-    </geometry>
-  </collision>
-</link>
-<link name="link4_1">
-  <inertial>
-    <origin xyz="-0.00473855751324301 8.608301182447264e-06 -0.02657822907239915" rpy="0 0 0"/>
-    <mass value="0.15464443104629289"/>
-    <inertia ixx="2.4e-05" iyy="3.9e-05" izz="2.4e-05" ixy="0.0" iyz="0.0" ixz="-3e-06"/>
-  </inertial>
-  <visual>
-    <origin xyz="-0.000175 -0.105258 -0.167394" rpy="0 0 0"/>
-    <geometry>
-      <mesh filename="file://$(find koch_description)/meshes/link4_1.stl" scale="0.001 0.001 0.001"/>
-    </geometry>
-    <material name="silver"/>
-  </visual>
-  <collision>
-    <origin xyz="-0.000175 -0.105258 -0.167394" rpy="0 0 0"/>
-    <geometry>
-      <mesh filename="file://$(find koch_description)/meshes/link4_1.stl" scale="0.001 0.001 0.001"/>
-    </geometry>
-  </collision>
-</link>
-<link name="gripper_static_1">
-  <inertial>
-    <origin xyz="0.005441113698877747 0.00011563276687967528 -0.019052234932530082" rpy="0 0 0"/>
-    <mass value="0.23008611256824127"/>
-    <inertia ixx="6.9e-05" iyy="8.4e-05" izz="4.3e-05" ixy="-0.0" iyz="0.0" ixz="1.8e-05"/>
-  </inertial>
-  <visual>
-    <origin xyz="-0.001528 -0.105265 -0.122394" rpy="0 0 0"/>
-    <geometry>
-      <mesh filename="file://$(find koch_description)/meshes/gripper_static_1.stl" scale="0.001 0.001 0.001"/>
-    </geometry>
-    <material name="silver"/>
-  </visual>
-  <collision>
-    <origin xyz="-0.001528 -0.105265 -0.122394" rpy="0 0 0"/>
-    <geometry>
-      <mesh filename="file://$(find koch_description)/meshes/gripper_static_1.stl" scale="0.001 0.001 0.001"/>
-    </geometry>
-  </collision>
-</link>
-<link name="gripper_moving_1">
-  <inertial>
-    <origin xyz="0.0010956016218150169 0.00031090398683926435 -0.02511314835420593" rpy="0 0 0"/>
-    <mass value="0.10060550172576842"/>
-    <inertia ixx="2.7e-05" iyy="1.9e-05" izz="1.2e-05" ixy="-0.0" iyz="0.0" ixz="2e-06"/>
-  </inertial>
-  <visual>
-    <origin xyz="0.005872 -0.105015 -0.109244" rpy="0 0 0"/>
-    <geometry>
-      <mesh filename="file://$(find koch_description)/meshes/gripper_moving_1.stl" scale="0.001 0.001 0.001"/>
-    </geometry>
-    <material name="silver"/>
-  </visual>
-  <collision>
-    <origin xyz="0.005872 -0.105015 -0.109244" rpy="0 0 0"/>
-    <geometry>
-      <mesh filename="file://$(find koch_description)/meshes/gripper_moving_1.stl" scale="0.001 0.001 0.001"/>
-    </geometry>
-  </collision>
-</link>
-<joint name="joint1" type="continuous">
-  <origin xyz="0.0 0.0 0.039" rpy="0 0 0"/>
-  <parent link="base_link"/>
-  <child link="link1_1"/>
-  <axis xyz="0.0 0.0 1.0"/>
-</joint>
-<joint name="joint2" type="continuous">
-  <origin xyz="-0.0002 -0.0 0.0173" rpy="0 0 0"/>
-  <parent link="link1_1"/>
-  <child link="link2_1"/>
-  <axis xyz="-1.0 -0.0 0.0"/>
-</joint>
-<joint name="joint3" type="continuous">
-  <origin xyz="0.00025 0.014791 0.108347" rpy="0 0 0"/>
-  <parent link="link2_1"/>
-  <child link="link3_1"/>
-  <axis xyz="1.0 0.0 0.0"/>
-</joint>
-<joint name="joint4" type="continuous">
-  <origin xyz="0.000125 0.090467 0.002747" rpy="0 0 0"/>
-  <parent link="link3_1"/>
-  <child link="link4_1"/>
-  <axis xyz="1.0 0.0 0.0"/>
-</joint>
-<joint name="joint5" type="continuous">
-  <origin xyz="0.001353 7e-06 -0.045" rpy="0 0 0"/>
-  <parent link="link4_1"/>
-  <child link="gripper_static_1"/>
-  <axis xyz="0.0 0.0 -1.0"/>
-</joint>
-<joint name="joint_gripper" type="continuous">
-  <origin xyz="-0.0074 -0.00025 -0.01315" rpy="0 0 0"/>
-  <parent link="gripper_static_1"/>
-  <child link="gripper_moving_1"/>
-  <axis xyz="-0.0 -1.0 -0.0"/>
-</joint>
+  <xacro:include filename="$(find koch_description)/urdf/materials.xacro" />
+  <xacro:include filename="$(find koch_description)/urdf/koch.trans" />
+  <xacro:include filename="$(find koch_description)/urdf/koch.gazebo" />
+  <link name="base_link">
+    <inertial>
+      <origin xyz="-0.00017023202404845418 -0.021341439639662032 0.014423161616418092" rpy="0 0 0"/>
+      <mass value="0.5164575020815119"/>
+      <inertia ixx="0.000304" iyy="0.000283" izz="0.000441" ixy="-2e-06" iyz="-6.2e-05" ixz="-1e-06"/>
+    </inertial>
+    <visual>
+      <origin xyz="0 0 0" rpy="0 0 0"/>
+      <geometry>
+        <mesh filename="file://$(find koch_description)/meshes/base_link.stl" scale="0.001 0.001 0.001"/>
+      </geometry>
+      <material name="silver"/>
+    </visual>
+    <collision>
+      <origin xyz="0 0 0" rpy="0 0 0"/>
+      <geometry>
+        <mesh filename="file://$(find koch_description)/meshes/base_link.stl" scale="0.001 0.001 0.001"/>
+      </geometry>
+    </collision>
+  </link>
+  <link name="link1_1">
+    <inertial>
+      <origin xyz="-0.0006216635769899589 -0.011914175885676576 0.015400174574576098" rpy="0 0 0"/>
+      <mass value="0.3956063453928257"/>
+      <inertia ixx="0.000112" iyy="7.5e-05" izz="0.000123" ixy="0.0" iyz="-1e-06" ixz="0.0"/>
+    </inertial>
+    <visual>
+      <origin xyz="-0.0 -0.0 -0.039" rpy="0 0 0"/>
+      <geometry>
+        <mesh filename="file://$(find koch_description)/meshes/link1_1.stl" scale="0.001 0.001 0.001"/>
+      </geometry>
+      <material name="silver"/>
+    </visual>
+    <collision>
+      <origin xyz="-0.0 -0.0 -0.039" rpy="0 0 0"/>
+      <geometry>
+        <mesh filename="file://$(find koch_description)/meshes/link1_1.stl" scale="0.001 0.001 0.001"/>
+      </geometry>
+    </collision>
+  </link>
+  <link name="link2_1">
+    <inertial>
+      <origin xyz="0.00015778948024297947 -0.0012168309893684582 0.07161179945761596" rpy="0 0 0"/>
+      <mass value="0.3916070272991037"/>
+      <inertia ixx="0.00052" iyy="0.000534" izz="8.4e-05" ixy="-1e-06" iyz="-3.7e-05" ixz="-2e-06"/>
+    </inertial>
+    <visual>
+      <origin xyz="0.0002 0.0 -0.0563" rpy="0 0 0"/>
+      <geometry>
+        <mesh filename="file://$(find koch_description)/meshes/link2_1.stl" scale="0.001 0.001 0.001"/>
+      </geometry>
+      <material name="silver"/>
+    </visual>
+    <collision>
+      <origin xyz="0.0002 0.0 -0.0563" rpy="0 0 0"/>
+      <geometry>
+        <mesh filename="file://$(find koch_description)/meshes/link2_1.stl" scale="0.001 0.001 0.001"/>
+      </geometry>
+    </collision>
+  </link>
+  <link name="link3_1">
+    <inertial>
+      <origin xyz="7.243666489899892e-05 0.05069893196527342 0.002850799344132765" rpy="0 0 0"/>
+      <mass value="0.4404689720232285"/>
+      <inertia ixx="0.000302" iyy="5.5e-05" izz="0.000322" ixy="-1e-06" iyz="-0.0" ixz="0.0"/>
+    </inertial>
+    <visual>
+      <origin xyz="-5e-05 -0.014791 -0.164647" rpy="0 0 0"/>
+      <geometry>
+        <mesh filename="file://$(find koch_description)/meshes/link3_1.stl" scale="0.001 0.001 0.001"/>
+      </geometry>
+      <material name="silver"/>
+    </visual>
+    <collision>
+      <origin xyz="-5e-05 -0.014791 -0.164647" rpy="0 0 0"/>
+      <geometry>
+        <mesh filename="file://$(find koch_description)/meshes/link3_1.stl" scale="0.001 0.001 0.001"/>
+      </geometry>
+    </collision>
+  </link>
+  <link name="link4_1">
+    <inertial>
+      <origin xyz="-0.00473855751324301 8.608301182447264e-06 -0.02657822907239915" rpy="0 0 0"/>
+      <mass value="0.15464443104629289"/>
+      <inertia ixx="2.4e-05" iyy="3.9e-05" izz="2.4e-05" ixy="0.0" iyz="0.0" ixz="-3e-06"/>
+    </inertial>
+    <visual>
+      <origin xyz="-0.000175 -0.105258 -0.167394" rpy="0 0 0"/>
+      <geometry>
+        <mesh filename="file://$(find koch_description)/meshes/link4_1.stl" scale="0.001 0.001 0.001"/>
+      </geometry>
+      <material name="silver"/>
+    </visual>
+    <collision>
+      <origin xyz="-0.000175 -0.105258 -0.167394" rpy="0 0 0"/>
+      <geometry>
+        <mesh filename="file://$(find koch_description)/meshes/link4_1.stl" scale="0.001 0.001 0.001"/>
+      </geometry>
+    </collision>
+  </link>
+  <link name="gripper_static_1">
+    <inertial>
+      <origin xyz="0.005441113698877747 0.00011563276687967528 -0.019052234932530082" rpy="0 0 0"/>
+      <mass value="0.23008611256824127"/>
+      <inertia ixx="6.9e-05" iyy="8.4e-05" izz="4.3e-05" ixy="-0.0" iyz="0.0" ixz="1.8e-05"/>
+    </inertial>
+    <visual>
+      <origin xyz="-0.001528 -0.105265 -0.122394" rpy="0 0 0"/>
+      <geometry>
+        <mesh filename="file://$(find koch_description)/meshes/gripper_static_1.stl" scale="0.001 0.001 0.001"/>
+      </geometry>
+      <material name="silver"/>
+    </visual>
+    <collision>
+      <origin xyz="-0.001528 -0.105265 -0.122394" rpy="0 0 0"/>
+      <geometry>
+        <mesh filename="file://$(find koch_description)/meshes/gripper_static_1.stl" scale="0.001 0.001 0.001"/>
+      </geometry>
+    </collision>
+  </link>
+  <link name="gripper_moving_1">
+    <inertial>
+      <origin xyz="0.0010956016218150169 0.00031090398683926435 -0.02511314835420593" rpy="0 0 0"/>
+      <mass value="0.10060550172576842"/>
+      <inertia ixx="2.7e-05" iyy="1.9e-05" izz="1.2e-05" ixy="-0.0" iyz="0.0" ixz="2e-06"/>
+    </inertial>
+    <visual>
+      <origin xyz="0.005872 -0.105015 -0.109244" rpy="0 0 0"/>
+      <geometry>
+        <mesh filename="file://$(find koch_description)/meshes/gripper_moving_1.stl" scale="0.001 0.001 0.001"/>
+      </geometry>
+      <material name="silver"/>
+    </visual>
+    <collision>
+      <origin xyz="0.005872 -0.105015 -0.109244" rpy="0 0 0"/>
+      <geometry>
+        <mesh filename="file://$(find koch_description)/meshes/gripper_moving_1.stl" scale="0.001 0.001 0.001"/>
+      </geometry>
+    </collision>
+  </link>
+  <joint name="joint1" type="continuous">
+    <origin xyz="0.0 0.0 0.039" rpy="0 0 0"/>
+    <parent link="base_link"/>
+    <child link="link1_1"/>
+    <axis xyz="0.0 0.0 1.0"/>
+  </joint>
+  <joint name="joint2" type="continuous">
+    <origin xyz="-0.0002 -0.0 0.0173" rpy="0 0 0"/>
+    <parent link="link1_1"/>
+    <child link="link2_1"/>
+    <axis xyz="-1.0 -0.0 0.0"/>
+  </joint>
+  <joint name="joint3" type="continuous">
+    <origin xyz="0.00025 0.014791 0.108347" rpy="0 0 0"/>
+    <parent link="link2_1"/>
+    <child link="link3_1"/>
+    <axis xyz="1.0 0.0 0.0"/>
+  </joint>
+  <joint name="joint4" type="continuous">
+    <origin xyz="0.000125 0.090467 0.002747" rpy="0 0 0"/>
+    <parent link="link3_1"/>
+    <child link="link4_1"/>
+    <axis xyz="1.0 0.0 0.0"/>
+  </joint>
+  <joint name="joint5" type="continuous">
+    <origin xyz="0.001353 7e-06 -0.045" rpy="0 0 0"/>
+    <parent link="link4_1"/>
+    <child link="gripper_static_1"/>
+    <axis xyz="0.0 0.0 -1.0"/>
+  </joint>
+  <joint name="joint_gripper" type="continuous">
+    <origin xyz="-0.0074 -0.00025 -0.01315" rpy="0 0 0"/>
+    <parent link="gripper_static_1"/>
+    <child link="gripper_moving_1"/>
+    <axis xyz="-0.0 -1.0 -0.0"/>
+  </joint>
+  <ros2_control name="koch_ros2_control" type="system">
+    <hardware>
+      <plugin>dynamixel_hardware/DynamixelHardware</plugin>
+      <param name="usb_port">/dev/ttyACM0</param>
+      <param name="baud_rate">1000000</param>
+      <!-- <param name="use_dummy">true</param> -->
+    </hardware>
+    <joint name="joint1">
+      <param name="id">1</param>
+      <command_interface name="position"/>
+      <command_interface name="velocity"/>
+      <state_interface name="position"/>
+      <state_interface name="velocity"/>
+      <state_interface name="effort"/>
+    </joint>
+    <joint name="joint2">
+      <param name="id">2</param>
+      <command_interface name="position"/>
+      <command_interface name="velocity"/>
+      <state_interface name="position"/>
+      <state_interface name="velocity"/>
+      <state_interface name="effort"/>
+    </joint>
+    <joint name="joint3">
+      <param name="id">3</param>
+      <command_interface name="position"/>
+      <command_interface name="velocity"/>
+      <state_interface name="position"/>
+      <state_interface name="velocity"/>
+      <state_interface name="effort"/>
+    </joint>
+    <joint name="joint4">
+      <param name="id">4</param>
+      <command_interface name="position"/>
+      <command_interface name="velocity"/>
+      <state_interface name="position"/>
+      <state_interface name="velocity"/>
+      <state_interface name="effort"/>
+    </joint>
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
Commit message: [koch_description] Add joint limits

File: koch_description/urdf/koch.xacro (robot description, xacro)
@@ -149,4 +149,5 @@
     <child link="link1_1"/>
     <axis xyz="0.0 0.0 1.0"/>
+    <limit lower="-3.141592653589793" upper="3.141592653589793" effort="1000.0" velocity="1.0"/>
   </joint>
   <joint name="joint2" type="continuous">
@@ -155,4 +156,5 @@
     <child link="link2_1"/>
     <axis xyz="-1.0 -0.0 0.0"/>
+    <limit lower="-1.5707963267948966" upper="1.5707963267948966" effort="1000.0" velocity="1.0"/>
   </joint>
   <joint name="joint3" type="continuous">
@@ -161,10 +163,12 @@
     <child link="link3_1"/>
     <axis xyz="1.0 0.0 0.0"/>
+    <limit lower="-1.48" upper="1.8" effort="1000.0" velocity="1.0"/>
   </joint>
   <joint name="joint4" type="continuous">
-    <origin xyz="0.000125 0.090467 0.002747" rpy="0 0 0"/>
+    <origin xyz="0.000125 0.090467 0.002747" rpy="1.57 0 0"/>
     <parent link="link3_1"/>
     <child link="link4_1"/>
     <axis xyz="1.0 0.0 0.0"/>
+    <limit lower="-2.0" upper="2.0" effort="1000.0" velocity="1.0"/>
   </joint>
   <joint name="joint5" type="continuous">
@@ -173,4 +177,5 @@
     <child link="gripper_static_1"/>
     <axis xyz="0.0 0.0 -1.0"/>
+    <limit lower="-3.141592653589793" upper="3.141592653589793" effort="1000.0" velocity="1.0"/>
   </joint>
   <joint name="joint_gripper" type="continuous">
@@ -179,4 +184,5 @@
     <child link="gripper_moving_1"/>
     <axis xyz="-0.0 -1.0 -0.0"/>
+    <limit lower="-0.5" upper="1.5707963267948966" effort="1000.0" velocity="1.0"/>
   </joint>
   <ros2_control name="koch_ros2_control" type="system">

Commit message: [koch_description] Fix the type of joints in xacro

File: koch_description/urdf/koch.xacro (robot description, xacro)
@@ -144,5 +144,5 @@
     </collision>
   </link>
-  <joint name="joint1" type="continuous">
+  <joint name="joint1" type="revolute">
     <origin xyz="0.0 0.0 0.039" rpy="0 0 0"/>
     <parent link="base_link"/>
@@ -151,5 +151,5 @@
     <limit lower="-3.141592653589793" upper="3.141592653589793" effort="1000.0" velocity="1.0"/>
   </joint>
-  <joint name="joint2" type="continuous">
+  <joint name="joint2" type="revolute">
     <origin xyz="-0.0002 -0.0 0.0173" rpy="0 0 0"/>
     <parent link="link1_1"/>
@@ -158,5 +158,5 @@
     <limit lower="-1.5707963267948966" upper="1.5707963267948966" effort="1000.0" velocity="1.0"/>
   </joint>
-  <joint name="joint3" type="continuous">
+  <joint name="joint3" type="revolute">
     <origin xyz="0.00025 0.014791 0.108347" rpy="0 0 0"/>
     <parent link="link2_1"/>
@@ -165,5 +165,5 @@
     <limit lower="-1.48" upper="1.8" effort="1000.0" velocity="1.0"/>
   </joint>
-  <joint name="joint4" type="continuous">
+  <joint name="joint4" type="revolute">
     <origin xyz="0.000125 0.090467 0.002747" rpy="1.57 0 0"/>
     <parent link="link3_1"/>
@@ -172,5 +172,5 @@
     <limit lower="-2.0" upper="2.0" effort="1000.0" velocity="1.0"/>
   </joint>
-  <joint name="joint5" type="continuous">
+  <joint name="joint5" type="revolute">
     <origin xyz="0.001353 7e-06 -0.045" rpy="0 0 0"/>
     <parent link="link4_1"/>
@@ -179,5 +179,5 @@
     <limit lower="-3.141592653589793" upper="3.141592653589793" effort="1000.0" velocity="1.0"/>
   </joint>
-  <joint name="joint_gripper" type="continuous">
+  <joint name="joint_gripper" type="revolute">
     <origin xyz="-0.0074 -0.00025 -0.01315" rpy="0 0 0"/>
     <parent link="gripper_static_1"/>

Commit message: [koch_description] Fix the kinematics and visualization for koch v1.1 robot
https://github.com/jess-moss/koch-v1-1

File: koch_description/urdf/koch.xacro (robot description, xacro)
@@ -91,5 +91,5 @@
     </inertial>
     <visual>
-      <origin xyz="-0.000175 -0.105258 -0.167394" rpy="0 0 0"/>
+      <origin xyz="-0.000175 0.105258 -0.167394" rpy="0 0 ${pi}"/>
       <geometry>
         <mesh filename="file://$(find koch_description)/meshes/link4_1.stl" scale="0.001 0.001 0.001"/>
@@ -98,5 +98,5 @@
     </visual>
     <collision>
-      <origin xyz="-0.000175 -0.105258 -0.167394" rpy="0 0 0"/>
+      <origin xyz="-0.000175 0.105258 -0.167394" rpy="0 0 ${pi}"/>
       <geometry>
         <mesh filename="file://$(find koch_description)/meshes/link4_1.stl" scale="0.001 0.001 0.001"/>
@@ -149,5 +149,5 @@
     <child link="link1_1"/>
     <axis xyz="0.0 0.0 1.0"/>
-    <limit lower="-3.141592653589793" upper="3.141592653589793" effort="1000.0" velocity="1.0"/>
+    <limit lower="-${pi}" upper="${pi}" effort="1000.0" velocity="1.0"/>
   </joint>
   <joint name="joint2" type="revolute">
@@ -156,5 +156,5 @@
     <child link="link2_1"/>
     <axis xyz="-1.0 -0.0 0.0"/>
-    <limit lower="-1.5707963267948966" upper="1.5707963267948966" effort="1000.0" velocity="1.0"/>
+    <limit lower="-${pi/2}" upper="${pi/2}" effort="1000.0" velocity="1.0"/>
   </joint>
   <joint name="joint3" type="revolute">
@@ -173,9 +173,9 @@
   </joint>
   <joint name="joint5" type="revolute">
-    <origin xyz="0.001353 7e-06 -0.045" rpy="0 0 0"/>
+    <origin xyz="0.001353 7e-06 -0.045" rpy="0 0 ${pi}"/>
     <parent link="link4_1"/>
     <child link="gripper_static_1"/>
     <axis xyz="0.0 0.0 -1.0"/>
-    <limit lower="-3.141592653589793" upper="3.141592653589793" effort="1000.0" velocity="1.0"/>
+    <limit lower="-${pi}" upper="${pi}" effort="1000.0" velocity="1.0"/>
   </joint>
   <joint name="joint_gripper" type="revolute">
@@ -183,6 +183,6 @@
     <parent link="gripper_static_1"/>
     <child link="gripper_moving_1"/>
-    <axis xyz="-0.0 -1.0 -0.0"/>
-    <limit lower="-0.5" upper="1.5707963267948966" effort="1000.0" velocity="1.0"/>
+    <axis xyz="-0.0 1.0 -0.0"/>
+    <limit lower="-0.5" upper="${pi/2}" effort="1000.0" velocity="1.0"/>
   </joint>
   <ros2_control name="koch_ros2_control" type="system">
