Commit message: feat: default Koch control to the maintained ROBOTIS driver
Select robotis, legacy or mock in xacro and all control launches, with
explicit per-arm ports. Preserve the passive leader and signed legacy
effort convention; use the e-Manual velocity scale. Keep legacy rollback.

Exercise the official 1.5.1 plugin and SDK 4.0.3 on isolated pty buses:
startup ordering, refusal, units, leader states, read faults, Fast Bulk
fallback, custom controller behavior and all three mock launches.

Use the approved 500 ms timeout: unsupported Fast Bulk needs about
355 ms to fall back; 250 ms failed. Document upstream per-servo torque
preflight and partial mode writes on refusal, without hiding them.

Three full colcon runs pass all new tests. The same two pre-existing
lint failures remain (99 flake8 diagnostics, three copyright omissions).
Both legacy renders match main before the later gain improvements.
No physical serial devices were opened.

File: koch_description/urdf/koch.xacro (robot description, xacro)
@@ -1,4 +1,7 @@
 <?xml version="1.0" ?>
 <robot name="koch" xmlns:xacro="http://www.ros.org/wiki/xacro">
+  <xacro:arg name="hardware" default="robotis"/>
+  <xacro:arg name="follower_port" default="/dev/ttyACM0"/>
+  <xacro:arg name="leader_port" default="/dev/ttyACM1"/>
   <xacro:include filename="$(find koch_description)/urdf/materials.xacro" />
   <xacro:include filename="$(find koch_description)/urdf/koch.trans" />
@@ -11,5 +14,5 @@
   <xacro:configure_transmissions prefix="follower_"/>
   <link name="base_link"/>
-  <xacro:koch_follower parent_link="base_link" xyz="-0.2 0 0" />
-  <xacro:koch_leader parent_link="base_link" xyz="0.2 0 0" />
+  <xacro:koch_follower hardware="$(arg hardware)" port="$(arg follower_port)" parent_link="base_link" xyz="-0.2 0 0" />
+  <xacro:koch_leader hardware="$(arg hardware)" port="$(arg leader_port)" parent_link="base_link" xyz="0.2 0 0" />
 </robot>

File: koch_description/urdf/koch_follower.xacro (robot description, xacro)
@@ -1,5 +1,6 @@
 <?xml version="1.0" ?>
 <robot xmlns:xacro="http://www.ros.org/wiki/xacro">
-  <xacro:macro name="koch_follower" params="parent_link:='' xyz:='0 0 0' rpy:='0 0 0'" >
+  <xacro:include filename="$(find koch_description)/urdf/koch_hardware.xacro"/>
+  <xacro:macro name="koch_follower" params="parent_link:='' xyz:='0 0 0' rpy:='0 0 0' hardware:='robotis' port:='/dev/ttyACM0'" >
     <xacro:unless value="${parent_link == ''}">
       <joint name="follower_${parent_link}_joint" type="fixed">
@@ -197,8 +198,9 @@
       <origin rpy="0 ${pi} 0" xyz="0.011 0 -0.052"/>
     </joint>
+    <xacro:if value="${hardware == 'legacy'}">
     <ros2_control name="koch_follower_ros2_control" type="system">
       <hardware>
         <plugin>dynamixel_hardware/DynamixelHardware</plugin>
-        <param name="usb_port">/dev/ttyACM0</param>
+        <param name="usb_port">${port}</param>
         <param name="baud_rate">1000000</param>
         <!-- <param name="enable_torque">false</param> -->
@@ -254,4 +256,8 @@
       </joint>
     </ros2_control>
+    </xacro:if>
+    <xacro:unless value="${hardware == 'legacy'}">
+      <xacro:koch_hardware arm="follower" hardware="${hardware}" port="${port}"/>
+    </xacro:unless>
   </xacro:macro>
 </robot>

File: koch_description/urdf/koch_follower_standalone.xacro (robot description, xacro)
@@ -1,4 +1,6 @@
 <?xml version="1.0" ?>
 <robot name="koch" xmlns:xacro="http://www.ros.org/wiki/xacro">
+  <xacro:arg name="hardware" default="robotis"/>
+  <xacro:arg name="follower_port" default="/dev/ttyACM0"/>
   <xacro:include filename="$(find koch_description)/urdf/materials.xacro" />
   <xacro:include filename="$(find koch_description)/urdf/koch.trans" />
@@ -8,4 +10,4 @@
   <xacro:configure_transmissions prefix="follower_"/>
   <link name="base_link"/>
-  <xacro:koch_follower parent_link="base_link" xyz="0 0 0" />
+  <xacro:koch_follower hardware="$(arg hardware)" port="$(arg follower_port)" parent_link="base_link" xyz="0 0 0" />
 </robot>

File: koch_description/urdf/koch_leader.xacro (robot description, xacro)
@@ -1,5 +1,6 @@
 <?xml version="1.0" ?>
 <robot xmlns:xacro="http://www.ros.org/wiki/xacro">
-  <xacro:macro name="koch_leader" params="parent_link:='' xyz:='0 0 0' rpy:='0 0 0'" >
+  <xacro:include filename="$(find koch_description)/urdf/koch_hardware.xacro"/>
+  <xacro:macro name="koch_leader" params="parent_link:='' xyz:='0 0 0' rpy:='0 0 0' hardware:='robotis' port:='/dev/ttyACM1'" >
     <xacro:unless value="${parent_link == ''}">
       <joint name="$leader_{parent_link}_joint" type="fixed">
@@ -191,8 +192,9 @@
       <limit lower="-${pi}" upper="${pi}" effort="1000.0" velocity="10.0"/>
     </joint>
+    <xacro:if value="${hardware == 'legacy'}">
     <ros2_control name="koch_leader_ros2_control" type="system">
       <hardware>
         <plugin>dynamixel_hardware/DynamixelHardware</plugin>
-        <param name="usb_port">/dev/ttyACM1</param>
+        <param name="usb_port">${port}</param>
         <param name="baud_rate">1000000</param>
         <param name="enable_torque">false</param>
@@ -248,4 +250,8 @@
       </joint>
     </ros2_control>
+    </xacro:if>
+    <xacro:unless value="${hardware == 'legacy'}">
+      <xacro:koch_hardware arm="leader" hardware="${hardware}" port="${port}"/>
+    </xacro:unless>
   </xacro:macro>
 </robot>
