Commit message: [koch_description] Add the leader arm with disabled torque

File: koch_description/urdf/koch_leader.xacro (robot description, xacro)
@@ -1,13 +1,13 @@
 <?xml version="1.0" ?>
 <robot xmlns:xacro="http://www.ros.org/wiki/xacro">
-  <xacro:macro name="koch_follower" params="parent_link:='' xyz:='0 0 0' rpy:='0 0 0'" >
+  <xacro:macro name="koch_leader" params="parent_link:='' xyz:='0 0 0' rpy:='0 0 0'" >
     <xacro:unless value="${parent_link == ''}">
-      <joint name="follower_${parent_link}_joint" type="fixed">
+      <joint name="$leader_{parent_link}_joint" type="fixed">
         <parent link="${parent_link}"/>
-        <child link="follower_base_link"/>
+        <child link="leader_base_link"/>
         <origin rpy="${rpy}" xyz="${xyz}"/>
       </joint>
     </xacro:unless>
-    <link name="follower_base_link">
+    <link name="leader_base_link">
       <inertial>
         <origin xyz="-0.00017023202404845418 -0.021341439639662032 0.014423161616418092" rpy="0 0 0"/>
@@ -29,5 +29,5 @@
       </collision>
     </link>
-    <link name="follower_link1_1">
+    <link name="leader_link1_1">
       <inertial>
         <origin xyz="-0.0006216635769899589 -0.011914175885676576 0.015400174574576098" rpy="0 0 0"/>
@@ -49,5 +49,5 @@
       </collision>
     </link>
-    <link name="follower_link2_1">
+    <link name="leader_link2_1">
       <inertial>
         <origin xyz="0.00015778948024297947 -0.0012168309893684582 0.07161179945761596" rpy="0 0 0"/>
@@ -69,5 +69,5 @@
       </collision>
     </link>
-    <link name="follower_link3_1">
+    <link name="leader_link3_1">
       <inertial>
         <origin xyz="7.243666489899892e-05 0.05069893196527342 0.002850799344132765" rpy="0 0 0"/>
@@ -89,5 +89,5 @@
       </collision>
     </link>
-    <link name="follower_link4_1">
+    <link name="leader_link4_1">
       <inertial>
         <origin xyz="-0.00473855751324301 8.608301182447264e-06 -0.02657822907239915" rpy="0 0 0"/>
@@ -109,5 +109,5 @@
       </collision>
     </link>
-    <link name="follower_gripper_static_1">
+    <link name="leader_gripper_static_1">
       <inertial>
         <origin xyz="0.005441113698877747 0.00011563276687967528 -0.019052234932530082" rpy="0 0 0"/>
@@ -129,5 +129,5 @@
       </collision>
     </link>
-    <link name="follower_gripper_moving_1">
+    <link name="leader_gripper_moving_1">
       <inertial>
         <origin xyz="0.0010956016218150169 0.00031090398683926435 -0.02511314835420593" rpy="0 0 0"/>
@@ -149,55 +149,55 @@
       </collision>
     </link>
-    <joint name="follower_joint1" type="revolute">
-      <origin xyz="0.0 0.0 0.039" rpy="0 0 0"/>
-      <parent link="follower_base_link"/>
-      <child link="follower_link1_1"/>
+    <joint name="leader_joint1" type="revolute">
+      <origin xyz="0.0 0.0 0.039" rpy="0 0 ${pi}"/>
+      <parent link="leader_base_link"/>
+      <child link="leader_link1_1"/>
       <axis xyz="0.0 0.0 1.0"/>
       <limit lower="-${pi}" upper="${pi}" effort="1000.0" velocity="1.0"/>
     </joint>
-    <joint name="follower_joint2" type="revolute">
+    <joint name="leader_joint2" type="revolute">
       <origin xyz="-0.0002 -0.0 0.0173" rpy="0 0 0"/>
-      <parent link="follower_link1_1"/>
-      <child link="follower_link2_1"/>
+      <parent link="leader_link1_1"/>
+      <child link="leader_link2_1"/>
       <axis xyz="-1.0 -0.0 0.0"/>
       <limit lower="-${pi/2}" upper="${pi/2}" effort="1000.0" velocity="1.0"/>
     </joint>
-    <joint name="follower_joint3" type="revolute">
+    <joint name="leader_joint3" type="revolute">
       <origin xyz="0.00025 0.014791 0.108347" rpy="0 0 0"/>
-      <parent link="follower_link2_1"/>
-      <child link="follower_link3_1"/>
-      <axis xyz="1.0 0.0 0.0"/>
+      <parent link="leader_link2_1"/>
+      <child link="leader_link3_1"/>
+      <axis xyz="-1.0 0.0 0.0"/>
       <limit lower="-1.48" upper="1.8" effort="1000.0" velocity="1.0"/>
     </joint>
-    <joint name="follower_joint4" type="revolute">
+    <joint name="leader_joint4" type="revolute">
       <origin xyz="0.000125 0.090467 0.002747" rpy="1.57 0 0"/>
-      <parent link="follower_link3_1"/>
-      <child link="follower_link4_1"/>
+      <parent link="leader_link3_1"/>
+      <child link="leader_link4_1"/>
       <axis xyz="1.0 0.0 0.0"/>
       <limit lower="-2.0" upper="2.0" effort="1000.0" velocity="1.0"/>
     </joint>
-    <joint name="follower_joint5" type="revolute">
-      <origin xyz="0.001353 7e-06 -0.045" rpy="0 0 ${pi}"/>
-      <parent link="follower_link4_1"/>
-      <child link="follower_gripper_static_1"/>
+    <joint name="leader_joint5" type="revolute">
+      <origin xyz="0.001353 7e-06 -0.045" rpy="0 0 0"/>
+      <parent link="leader_link4_1"/>
+      <child link="leader_gripper_static_1"/>
       <axis xyz="0.0 0.0 -1.0"/>
       <limit lower="-${pi}" upper="${pi}" effort="1000.0" velocity="1.0"/>
     </joint>
-    <joint name="follower_joint_gripper" type="revolute">
+    <joint name="leader_joint_gripper" type="revolute">
       <origin xyz="-0.0074 -0.00025 -0.01315" rpy="0 0 0"/>
-      <parent link="follower_gripper_static_1"/>
-      <child link="follower_gripper_moving_1"/>
+      <parent link="leader_gripper_static_1"/>
+      <child link="leader_gripper_moving_1"/>
       <axis xyz="-0.0 1.0 -0.0"/>
       <limit lower="-0.5" upper="${pi/2}" effort="1000.0" velocity="1.0"/>
     </joint>
-    <ros2_control name="koch_follower_ros2_control" type="system">
+    <ros2_control name="koch_leader_ros2_control" type="system">
       <hardware>
         <plugin>dynamixel_hardware/DynamixelHardware</plugin>
-        <param name="usb_port">/dev/ttyACM0</param>
+        <param name="usb_port">/dev/ttyACM1</param>
         <param name="baud_rate">1000000</param>
-        <!-- <param name="enable_torque">false</param> -->
+        <param name="enable_torque">false</param>
         <!-- <param name="use_dummy">true</param> -->
       </hardware>
-      <joint name="follower_joint1">
+      <joint name="leader_joint1">
         <param name="id">1</param>
         <command_interface name="position"/>
@@ -207,5 +207,5 @@
         <state_interface name="effort"/>
       </joint>
-      <joint name="follower_joint2">
+      <joint name="leader_joint2">
         <param name="id">2</param>
         <command_interface name="position"/>
@@ -215,5 +215,5 @@
         <state_interface name="effort"/>
       </joint>
-      <joint name="follower_joint3">
+      <joint name="leader_joint3">
         <param name="id">3</param>
         <command_interface name="position"/>
@@ -223,5 +223,5 @@
         <state_interface name="effort"/>
       </joint>
-      <joint name="follower_joint4">
+      <joint name="leader_joint4">
         <param name="id">4</param>
         <command_interface name="position"/>
@@ -231,5 +231,5 @@
         <state_interface name="effort"/>
       </joint>
-      <joint name="follower_joint5">
+      <joint name="leader_joint5">
         <param name="id">5</param>
         <command_interface name="position"/>
@@ -239,5 +239,5 @@
         <state_interface name="effort"/>
       </joint>
-      <joint name="follower_joint_gripper">
+      <joint name="leader_joint_gripper">
         <param name="id">6</param>
         <command_interface name="position"/>
