Commit message: [koch_description] Make the namings clear for the follower robot

File: koch_description/urdf/koch_follower.xacro (robot description, xacro)
@@ -1,8 +1,8 @@
 <?xml version="1.0" ?>
-<robot name="koch" xmlns:xacro="http://www.ros.org/wiki/xacro">
+<robot name="koch_follower" xmlns:xacro="http://www.ros.org/wiki/xacro">
   <xacro:include filename="$(find koch_description)/urdf/materials.xacro" />
-  <xacro:include filename="$(find koch_description)/urdf/koch.trans" />
-  <xacro:include filename="$(find koch_description)/urdf/koch.gazebo" />
-  <link name="base_link">
+  <xacro:include filename="$(find koch_description)/urdf/koch_follower.trans" />
+  <xacro:include filename="$(find koch_description)/urdf/koch_follower.gazebo" />
+  <link name="follower_base_link">
     <inertial>
       <origin xyz="-0.00017023202404845418 -0.021341439639662032 0.014423161616418092" rpy="0 0 0"/>
@@ -24,5 +24,5 @@
     </collision>
   </link>
-  <link name="link1_1">
+  <link name="follower_link1_1">
     <inertial>
       <origin xyz="-0.0006216635769899589 -0.011914175885676576 0.015400174574576098" rpy="0 0 0"/>
@@ -44,5 +44,5 @@
     </collision>
   </link>
-  <link name="link2_1">
+  <link name="follower_link2_1">
     <inertial>
       <origin xyz="0.00015778948024297947 -0.0012168309893684582 0.07161179945761596" rpy="0 0 0"/>
@@ -64,5 +64,5 @@
     </collision>
   </link>
-  <link name="link3_1">
+  <link name="follower_link3_1">
     <inertial>
       <origin xyz="7.243666489899892e-05 0.05069893196527342 0.002850799344132765" rpy="0 0 0"/>
@@ -84,5 +84,5 @@
     </collision>
   </link>
-  <link name="link4_1">
+  <link name="follower_link4_1">
     <inertial>
       <origin xyz="-0.00473855751324301 8.608301182447264e-06 -0.02657822907239915" rpy="0 0 0"/>
@@ -144,40 +144,40 @@
     </collision>
   </link>
-  <joint name="joint1" type="revolute">
+  <joint name="follower_joint1" type="revolute">
     <origin xyz="0.0 0.0 0.039" rpy="0 0 0"/>
-    <parent link="base_link"/>
-    <child link="link1_1"/>
+    <parent link="follower_base_link"/>
+    <child link="follower_link1_1"/>
     <axis xyz="0.0 0.0 1.0"/>
     <limit lower="-${pi}" upper="${pi}" effort="1000.0" velocity="1.0"/>
   </joint>
-  <joint name="joint2" type="revolute">
+  <joint name="follower_joint2" type="revolute">
     <origin xyz="-0.0002 -0.0 0.0173" rpy="0 0 0"/>
-    <parent link="link1_1"/>
-    <child link="link2_1"/>
+    <parent link="follower_link1_1"/>
+    <child link="follower_link2_1"/>
     <axis xyz="-1.0 -0.0 0.0"/>
     <limit lower="-${pi/2}" upper="${pi/2}" effort="1000.0" velocity="1.0"/>
   </joint>
-  <joint name="joint3" type="revolute">
+  <joint name="follower_joint3" type="revolute">
     <origin xyz="0.00025 0.014791 0.108347" rpy="0 0 0"/>
-    <parent link="link2_1"/>
-    <child link="link3_1"/>
+    <parent link="follower_link2_1"/>
+    <child link="follower_link3_1"/>
     <axis xyz="1.0 0.0 0.0"/>
     <limit lower="-1.48" upper="1.8" effort="1000.0" velocity="1.0"/>
   </joint>
-  <joint name="joint4" type="revolute">
+  <joint name="follower_joint4" type="revolute">
     <origin xyz="0.000125 0.090467 0.002747" rpy="1.57 0 0"/>
-    <parent link="link3_1"/>
-    <child link="link4_1"/>
+    <parent link="follower_link3_1"/>
+    <child link="follower_link4_1"/>
     <axis xyz="1.0 0.0 0.0"/>
     <limit lower="-2.0" upper="2.0" effort="1000.0" velocity="1.0"/>
   </joint>
-  <joint name="joint5" type="revolute">
+  <joint name="follower_joint5" type="revolute">
     <origin xyz="0.001353 7e-06 -0.045" rpy="0 0 ${pi}"/>
-    <parent link="link4_1"/>
+    <parent link="follower_link4_1"/>
     <child link="gripper_static_1"/>
     <axis xyz="0.0 0.0 -1.0"/>
     <limit lower="-${pi}" upper="${pi}" effort="1000.0" velocity="1.0"/>
   </joint>
-  <joint name="joint_gripper" type="revolute">
+  <joint name="follower_joint_gripper" type="revolute">
     <origin xyz="-0.0074 -0.00025 -0.01315" rpy="0 0 0"/>
     <parent link="gripper_static_1"/>
@@ -191,7 +191,8 @@
       <param name="usb_port">/dev/ttyACM0</param>
       <param name="baud_rate">1000000</param>
+      <!-- <param name="enable_torque">false</param> -->
       <!-- <param name="use_dummy">true</param> -->
     </hardware>
-    <joint name="joint1">
+    <joint name="follower_joint1">
       <param name="id">1</param>
       <command_interface name="position"/>
@@ -201,5 +202,5 @@
       <state_interface name="effort"/>
     </joint>
-    <joint name="joint2">
+    <joint name="follower_joint2">
       <param name="id">2</param>
       <command_interface name="position"/>
@@ -209,5 +210,5 @@
       <state_interface name="effort"/>
     </joint>
-    <joint name="joint3">
+    <joint name="follower_joint3">
       <param name="id">3</param>
       <command_interface name="position"/>
@@ -217,5 +218,5 @@
       <state_interface name="effort"/>
     </joint>
-    <joint name="joint4">
+    <joint name="follower_joint4">
       <param name="id">4</param>
       <command_interface name="position"/>
@@ -225,5 +226,5 @@
       <state_interface name="effort"/>
     </joint>
-    <joint name="joint5">
+    <joint name="follower_joint5">
       <param name="id">5</param>
       <command_interface name="position"/>
@@ -233,5 +234,5 @@
       <state_interface name="effort"/>
     </joint>
-    <joint name="joint_gripper">
+    <joint name="follower_joint_gripper">
       <param name="id">6</param>
       <command_interface name="position"/>

Commit message: Add leader follower controller
https://github.com/Maverobot/koch_ros/issues/5

File: koch_description/urdf/koch_follower.xacro (robot description, xacro)
@@ -154,5 +154,5 @@
       <child link="follower_link1_1"/>
       <axis xyz="0.0 0.0 1.0"/>
-      <limit lower="-${pi}" upper="${pi}" effort="1000.0" velocity="1.0"/>
+      <limit lower="-${pi}" upper="${pi}" effort="1000.0" velocity="10.0"/>
     </joint>
     <joint name="follower_joint2" type="revolute">
@@ -161,5 +161,5 @@
       <child link="follower_link2_1"/>
       <axis xyz="-1.0 -0.0 0.0"/>
-      <limit lower="-${pi/2}" upper="${pi/2}" effort="1000.0" velocity="1.0"/>
+      <limit lower="-${pi/2}" upper="${pi/2}" effort="1000.0" velocity="10.0"/>
     </joint>
     <joint name="follower_joint3" type="revolute">
@@ -168,5 +168,5 @@
       <child link="follower_link3_1"/>
       <axis xyz="1.0 0.0 0.0"/>
-      <limit lower="-1.48" upper="1.8" effort="1000.0" velocity="1.0"/>
+      <limit lower="-1.48" upper="1.8" effort="1000.0" velocity="10.0"/>
     </joint>
     <joint name="follower_joint4" type="revolute">
@@ -175,5 +175,5 @@
       <child link="follower_link4_1"/>
       <axis xyz="1.0 0.0 0.0"/>
-      <limit lower="-2.0" upper="2.0" effort="1000.0" velocity="1.0"/>
+      <limit lower="-2.0" upper="2.0" effort="1000.0" velocity="10.0"/>
     </joint>
     <joint name="follower_joint5" type="revolute">
@@ -182,5 +182,5 @@
       <child link="follower_gripper_static_1"/>
       <axis xyz="0.0 0.0 -1.0"/>
-      <limit lower="-${pi}" upper="${pi}" effort="1000.0" velocity="1.0"/>
+      <limit lower="-${pi}" upper="${pi}" effort="1000.0" velocity="10.0"/>
     </joint>
     <joint name="follower_joint_gripper" type="revolute">
@@ -189,5 +189,5 @@
       <child link="follower_gripper_moving_1"/>
       <axis xyz="-0.0 1.0 -0.0"/>
-      <limit lower="-0.5" upper="${pi/2}" effort="1000.0" velocity="1.0"/>
+      <limit lower="-0.5" upper="${pi/2}" effort="1000.0" velocity="10.0"/>
     </joint>
     <ros2_control name="koch_follower_ros2_control" type="system">

File: koch_description/urdf/koch_leader.xacro (robot description, xacro)
@@ -154,5 +154,5 @@
       <child link="leader_link1_1"/>
       <axis xyz="0.0 0.0 1.0"/>
-      <limit lower="-${pi}" upper="${pi}" effort="1000.0" velocity="1.0"/>
+      <limit lower="-${pi}" upper="${pi}" effort="1000.0" velocity="10.0"/>
     </joint>
     <joint name="leader_joint2" type="revolute">
@@ -161,5 +161,5 @@
       <child link="leader_link2_1"/>
       <axis xyz="-1.0 -0.0 0.0"/>
-      <limit lower="-${pi/2}" upper="${pi/2}" effort="1000.0" velocity="1.0"/>
+      <limit lower="-${pi/2}" upper="${pi/2}" effort="1000.0" velocity="10.0"/>
     </joint>
     <joint name="leader_joint3" type="revolute">
@@ -168,5 +168,5 @@
       <child link="leader_link3_1"/>
       <axis xyz="-1.0 0.0 0.0"/>
-      <limit lower="-1.48" upper="1.8" effort="1000.0" velocity="1.0"/>
+      <limit lower="-1.48" upper="1.8" effort="1000.0" velocity="10.0"/>
     </joint>
     <joint name="leader_joint4" type="revolute">
@@ -175,5 +175,5 @@
       <child link="leader_link4_1"/>
       <axis xyz="1.0 0.0 0.0"/>
-      <limit lower="-2.0" upper="2.0" effort="1000.0" velocity="1.0"/>
+      <limit lower="-2.0" upper="2.0" effort="1000.0" velocity="10.0"/>
     </joint>
     <joint name="leader_joint5" type="revolute">
@@ -182,5 +182,5 @@
       <child link="leader_gripper_static_1"/>
       <axis xyz="0.0 0.0 -1.0"/>
-      <limit lower="-${pi}" upper="${pi}" effort="1000.0" velocity="1.0"/>
+      <limit lower="-${pi}" upper="${pi}" effort="1000.0" velocity="10.0"/>
     </joint>
     <joint name="leader_joint_gripper" type="revolute">
@@ -189,5 +189,5 @@
       <child link="leader_gripper_moving_1"/>
       <axis xyz="-0.0 1.0 -0.0"/>
-      <limit lower="-0.5" upper="${pi/2}" effort="1000.0" velocity="1.0"/>
+      <limit lower="-0.5" upper="${pi/2}" effort="1000.0" velocity="10.0"/>
     </joint>
     <ros2_control name="koch_leader_ros2_control" type="system">

Commit message: [koch_description] Relax the all joint limits to [-pi, pi]
Fixes: https://github.com/Maverobot/koch_ros/issues/8

File: koch_description/urdf/koch_follower.xacro (robot description, xacro)
@@ -161,5 +161,5 @@
       <child link="follower_link2_1"/>
       <axis xyz="-1.0 -0.0 0.0"/>
-      <limit lower="-${pi/2}" upper="${pi/2}" effort="1000.0" velocity="10.0"/>
+      <limit lower="-${pi}" upper="${pi}" effort="1000.0" velocity="10.0"/>
     </joint>
     <joint name="follower_joint3" type="revolute">
@@ -168,5 +168,5 @@
       <child link="follower_link3_1"/>
       <axis xyz="1.0 0.0 0.0"/>
-      <limit lower="-1.48" upper="1.8" effort="1000.0" velocity="10.0"/>
+      <limit lower="-${pi}" upper="${pi}" effort="1000.0" velocity="10.0"/>
     </joint>
     <joint name="follower_joint4" type="revolute">
@@ -175,5 +175,5 @@
       <child link="follower_link4_1"/>
       <axis xyz="1.0 0.0 0.0"/>
-      <limit lower="-2.0" upper="2.0" effort="1000.0" velocity="10.0"/>
+      <limit lower="-${pi}" upper="${pi}" effort="1000.0" velocity="10.0"/>
     </joint>
     <joint name="follower_joint5" type="revolute">
@@ -189,5 +189,5 @@
       <child link="follower_gripper_moving_1"/>
       <axis xyz="-0.0 1.0 -0.0"/>
-      <limit lower="-0.5" upper="${pi/2}" effort="1000.0" velocity="10.0"/>
+      <limit lower="-${pi}" upper="${pi}" effort="1000.0" velocity="10.0"/>
     </joint>
     <ros2_control name="koch_follower_ros2_control" type="system">

File: koch_description/urdf/koch_leader.xacro (robot description, xacro)
@@ -161,5 +161,5 @@
       <child link="leader_link2_1"/>
       <axis xyz="-1.0 -0.0 0.0"/>
-      <limit lower="-${pi/2}" upper="${pi/2}" effort="1000.0" velocity="10.0"/>
+      <limit lower="-${pi}" upper="${pi}" effort="1000.0" velocity="10.0"/>
     </joint>
     <joint name="leader_joint3" type="revolute">
@@ -168,5 +168,5 @@
       <child link="leader_link3_1"/>
       <axis xyz="-1.0 0.0 0.0"/>
-      <limit lower="-1.48" upper="1.8" effort="1000.0" velocity="10.0"/>
+      <limit lower="-${pi}" upper="${pi}" effort="1000.0" velocity="10.0"/>
     </joint>
     <joint name="leader_joint4" type="revolute">
@@ -175,5 +175,5 @@
       <child link="leader_link4_1"/>
       <axis xyz="1.0 0.0 0.0"/>
-      <limit lower="-2.0" upper="2.0" effort="1000.0" velocity="10.0"/>
+      <limit lower="-${pi}" upper="${pi}" effort="1000.0" velocity="10.0"/>
     </joint>
     <joint name="leader_joint5" type="revolute">
@@ -189,5 +189,5 @@
       <child link="leader_gripper_moving_1"/>
       <axis xyz="-0.0 1.0 -0.0"/>
-      <limit lower="-0.5" upper="${pi/2}" effort="1000.0" velocity="10.0"/>
+      <limit lower="-${pi}" upper="${pi}" effort="1000.0" velocity="10.0"/>
     </joint>
     <ros2_control name="koch_leader_ros2_control" type="system">

Commit message: [koch_controllers] Implement position forward kinematics for follower

File: koch_description/urdf/koch_follower.xacro (robot description, xacro)
@@ -149,4 +149,5 @@
       </collision>
     </link>
+    <link name="follower_gripper_tip"/>
     <joint name="follower_joint1" type="revolute">
       <origin xyz="0.0 0.0 0.039" rpy="0 0 0"/>
@@ -190,4 +191,9 @@
       <axis xyz="-0.0 1.0 -0.0"/>
       <limit lower="-${pi}" upper="${pi}" effort="1000.0" velocity="10.0"/>
+    </joint>
+    <joint name="follower_joint_gripper_tip" type="fixed">
+      <parent link="follower_gripper_moving_1"/>
+      <child link="follower_gripper_tip"/>
+      <origin rpy="0 ${pi} 0" xyz="0.011 0 -0.052"/>
     </joint>
     <ros2_control name="koch_follower_ros2_control" type="system">
