Commit message: fix(kinematics): use nominal 100.5 mm follower forearm
Correct the follower forearm using a ruler-supported nominal dimension.
This remains an experimental candidate, not confirmed physical ground
truth.

Derive the POE forearm contribution from each controller's actual robot
description so old frozen models retain their previous behavior.

Leave leader geometry, meshes and inertia unchanged. Collision accuracy
and the remaining calibration residuals are not validated here.

File: koch_description/urdf/koch_follower.xacro (robot description, xacro)
@@ -173,5 +173,5 @@
     </joint>
     <joint name="follower_joint4" type="revolute">
-      <origin xyz="0.000125 0.090467 0.002747" rpy="1.57 0 0"/>
+      <origin xyz="0.000125 0.100467 0.002747" rpy="1.57 0 0"/>
       <parent link="follower_link3_1"/>
       <child link="follower_link4_1"/>
